Commit message: working gs mini finger + franka

File: assets/TacSL_gym/urdf/gsmini_finger.urdf (robot description, URDF)
Before this commit: robot gelsight_finger, 5 links, 4 joints
Links:
- removed link camera_link
Joints:
- removed joint tactile_camera_joint

Commit message: gsmini works! calibration data seems weird

File: assets/TacSL_gym/urdf/gsmini_finger.urdf (robot description, URDF)
Before this commit: robot gelsight_finger, 4 links, 3 joints
Joints:
- joint elastomer_tip_joint: origin xyz=-0.00050001 -0.05975001 -0.01125 rpy=3.141592653589793 0 0 -> xyz=0.00050001 -0.01125 0.05975001 rpy=3.141592653589793 0 0
